File: Arm-EStop_Hardware/Arm-EStop_Hardware.kicad_pcb (KiCad board)
At the start: 2 copper layers, 208.3 x 76.2 mm, 132 parts, among them Q1 2N7002PW, Q2 2N7002PW, Q3 2N7002PW, Q4 2N7002PW, Q5 2N7002PW, Q6 IRLS3034-7P, Q7 IRLS3034-7P, Q8 2N7002PW, U1 ACS759ECB-200B-PFF-T, U10 E_STOP+LED, U11 TEMP_1, U12 FAN_4, U13 INA132, U14 INA132, U15 INA132, U16 OKI, U17 Indicator Comm, U18 OKI, U19 INA132, U2 FAN_1, U20 INA132, U21 TM4C129E_Launchpad, U3 INA132, U4 FAN_2, U5 BMS_Logic_Switch, U6 LT1910, U7 E_STOP, U8 FAN_3, U9 INA132

Commit message: started layout
Parts:
- removed B1: BUZZER_SMI_1324_TW_5V_2_R, MRDT_Devices:BUZZER_SMI_1324_TW_5V_2_R
- removed C10: 10u, Capacitor_SMD:C_1206_3216Metric_Pad1.42x1.75mm_HandSolder
- removed C11, C12, C13, C14, C15, C16, C5, C6, C7, C8, C9: 1u, Capacitor_SMD:C_0603_1608Metric_Pad1.05x0.95mm_HandSolder
- removed C17, C26: 22u 50V, Capacitor_THT:CP_Radial_D6.3mm_P2.50mm
- removed C18, C19, C20, C21, C27, C28, C29, C30: 10u, Capacitor_SMD:C_0603_1608Metric_Pad1.05x0.95mm_HandSolder
- removed C22, C31: 0.1u, Capacitor_SMD:C_0603_1608Metric_Pad1.05x0.95mm_HandSolder
- removed Conn3: AndersonPP, MRDT_Connectors:Anderson_2_Vertical_Sidy_by_Side
- removed D10: PACK_V_IND_LED_ORANGE, LED_SMD:LED_0603_1608Metric_Pad1.05x0.95mm_HandSolder
- removed D11: SW_IND_LED_BLUE, LED_SMD:LED_0603_1608Metric_Pad1.05x0.95mm_HandSolder
- removed D12, D13, D14, D15, D16, D17, D18, D19, D20, D22: D_Zener, Diode_SMD:D_SOD-323_HandSoldering
- removed D21: SW_ERR_LED_RED, LED_SMD:LED_0603_1608Metric_Pad1.05x0.95mm_HandSolder
- removed D23: FAN_PWR_LED_ORANGE, LED_SMD:LED_0603_1608Metric_Pad1.05x0.95mm_HandSolder
- removed D4, D5, D6, D7, D8: 7.5V, Diode_SMD:D_SOD-323_HandSoldering
- removed D9: LOG_PWR_LED, LED_SMD:LED_0603_1608Metric_Pad1.05x0.95mm_HandSolder
- removed G***: LOGO, BMS_Hardware:Brian_Dahlman_Sig_20.1mmX7.5mm
- removed G***: LOGO, MRDT_Silkscreens:MRDT_Logo_20mm
- removed G***: LOGO, MRDT_Silkscreens:Nothing_3mm_Cu
- removed G***: LOGO, MRDT_Silkscreens:2_Dahlbot_2.0
- removed G***: LOGO, MRDT_Silkscreens:zz_Valkyrie_Logo_Full_50mmx50mm
- removed Q3, Q4, Q5, Q8: 2N7002PW, TO_SOT_Packages_SMD:SOT-23_Handsoldering
- removed Q6, Q7: IRLS3034-7P, MRDT_Actives:IRLS3034_TO-263-7_P
- removed R10, R12, R20, R24: 100K, Resistor_SMD:R_0603_1608Metric_Pad1.05x0.95mm_HandSolder
- removed R11: 10K, Resistor_SMD:R_0603_1608Metric_Pad1.05x0.95mm_HandSolder
- removed R13, R16, R19, R23, R6, R7, R8, R9: 10k, Resistor_SMD:R_0603_1608Metric_Pad1.05x0.95mm_HandSolder
- removed R14: 1M, Resistor_SMD:R_0603_1608Metric_Pad1.05x0.95mm_HandSolder
- removed R15, R22: 100k, Resistor_SMD:R_0603_1608Metric_Pad1.05x0.95mm_HandSolder
- removed R17, R21, R30, R31, R32, R33, R34: 36.5k, Resistor_SMD:R_0603_1608Metric_Pad1.05x0.95mm_HandSolder
- removed R18: 4k, Resistor_SMD:R_0603_1608Metric_Pad1.05x0.95mm_HandSolder
- removed R25, R27, R28, R35: 500, Resistor_SMD:R_0603_1608Metric_Pad1.05x0.95mm_HandSolder
- removed R26: 1.5k, Resistor_SMD:R_0603_1608Metric_Pad1.05x0.95mm_HandSolder
- removed R29: 820, Resistor_SMD:R_0603_1608Metric_Pad1.05x0.95mm_HandSolder
- removed REF** (x4): 4_40_Hole, MRDT_Drill_Holes:4_40_Hole
- removed U10: E_STOP+LED, MRDT_Connectors:MOLEX_SL_04_Vertical
- removed U11: TEMP_1, MRDT_Connectors:MOLEX_SL_03_Vertical
- removed U12: FAN_4, MRDT_Connectors:MOLEX_SL_02_Vertical
- removed U13, U14, U15, U19, U20, U9: INA132, Package_SO:SO-8_5.3x6.2mm_P1.27mm
- removed U16, U18: OKI, MRDT_Devices:OKI_Horizontal
- removed U17: Indicator Comm, MRDT_Connectors:MOLEX_SL_03_Vertical
- removed U21: TM4C129E_Launchpad, MRDT_Shields:TM4C129E_Launchpad_FULL_SMD_TOP
- removed U6: LT1910, Housings_SOIC:SOIC-8_3.9x4.9mm_Pitch1.27mm
- removed U7: E_STOP, MRDT_Connectors:MOLEX_SL_02_Vertical
- removed U8: FAN_3, MRDT_Connectors:MOLEX_SL_02_Vertical
- removed V1, V2, V3: BATT_PWR_VIA, MRDT_Drill_Holes:BATT_PWR_VIA
- added F2: 5A, MRDT_Passives:ATC_Fuse_Block, F.Cu at (211.5, 38.1)
- added SW1: SW_Push_Open, Button_Switch_SMD:SW_SPST_TL3305A, F.Cu at (112.8, 108.2)
- C1, C2, C3, C4: value 1u -> 10u
- Conn1: value CHARGE_SENSE_BOTTOM -> AndersonPP; footprint MRDT_Connectors:MOLEX_SL_09_Vertical -> MRDT_Connectors:Anderson_2_Horizontal_Side_by_Side; moved to F.Cu
- Conn2: value CHARGE_SENSE_TOP -> AndersonPP; footprint MRDT_Connectors:MOLEX_SL_09_Vertical -> MRDT_Connectors:Anderson_3_Horizontal_Side_by_Side; moved to F.Cu
- D1, D2, D3: value 7.5V -> Green; footprint Diode_SMD:D_SOD-323_HandSoldering -> Diode_SMD:D_0603_1608Metric_Pad1.05x0.95mm_HandSolder
- F1: value PTC2920 -> 20A; footprint Fuse:Fuse_2920_7451Metric -> MRDT_Passives:ATC_Fuse_Block
- Q1, Q2: value 2N7002PW -> IRFS7437TRLPBFCT; footprint TO_SOT_Packages_SMD:SOT-23_Handsoldering -> Package_TO_SOT_SMD:TO-263-2
- R1, R3: value 10k -> 1K
- R2: value 36.5k -> 1K
- U1: value ACS759ECB-200B-PFF-T -> 3.3V; footprint MRDT_Sensors:ACS759ECB_PFF_Leadform_5pins -> MRDT_Devices:OKI_Horizontal
- U2: value FAN_1 -> LT1910; footprint MRDT_Connectors:MOLEX_SL_02_Vertical -> Package_SO:SOIC-8_3.9x4.9mm_P1.27mm; moved to F.Cu
- U3: value INA132 -> LT1910; footprint Package_SO:SO-8_5.3x6.2mm_P1.27mm -> Package_SO:SOIC-8_3.9x4.9mm_P1.27mm
- U4: value FAN_2 -> E_STOP; moved to F.Cu
- U5: value BMS_Logic_Switch -> E_STOP+LED; moved to F.Cu
- moved U4 205.8 mm to (266.7, 96.5)
- moved U2 139.5 mm to (177.6, 118.7)
- moved Q1 130.7 mm to (182.2, 33.0)
- moved U3 97.4 mm to (233.5, 106.0)
- moved C4 91.5 mm to (235.3, 101.6), turned to 180 degrees
- moved R5 88.2 mm to (232.0, 110.5), turned to 0 degrees
- moved U1 88.0 mm to (127.0, 67.3)
- moved U5 85.4 mm to (246.4, 88.9), turned to 0 degrees
- moved Q2 85.1 mm to (182.2, 45.7), turned to 180 degrees
- moved Conn2 83.4 mm to (224.5, 31.1)
- moved F1 71.9 mm to (211.5, 30.5), turned to 180 degrees
- moved Conn1 51.1 mm to (95.5, 60.1), turned to 0 degrees
- moved R4 41.2 mm to (176.1, 123.2), turned to 0 degrees
- moved C3 41.0 mm to (179.5, 114.3), turned to 180 degrees
- moved C1 39.5 mm to (130.4, 66.0), turned to 0 degrees
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Connections:
- C1 pad 1: GND -> V_In
- C1 pad 2: CELL_1 -> GND
- C2 pad 1: GND -> +3V3
- C2 pad 2: LOGIC_PWR -> GND
- C3 pad 1: GND -> V_In
- C3 pad 2: LOGIC_PWR -> GND
- C4 pad 1: GND -> V_In
- C4 pad 2: LOGIC_PWR -> GND
- Conn1 pad 1: CELL_1 -> GND
- Conn1 pad 2: CELL_2 -> V_In
- Conn2 pad 1: CELL_1 -> GND
- Conn2 pad 2: CELL_2 -> Net-(Conn2-Pad2)
- Conn2 pad 3: CELL_3 -> Net-(Conn2-Pad3)
- D1 pad 1: CELL_1 -> GND
- D1 pad 2: GND -> Net-(D1-Pad2)
- D2 pad 1: CELL_8 -> GND
- D2 pad 2: CELL_7 -> Net-(D2-Pad2)
- D3 pad 1: CELL_7 -> GND
- D3 pad 2: CELL_6 -> Net-(D3-Pad2)
- F1 pad 1: LOGIC_PWR -> Net-(Conn2-Pad3)
- F1 pad 2: Net-(F1-Pad2) -> V_Out_Act
- Q1 pad 1: FAN_CTL_1 -> E-Stop_Gate
- Q1 pad 2: GND -> V_In
- Q1 pad 3: Net-(Q1-Pad3) -> V_Out_Act
- Q2 pad 1: LOGIC_SWITCH -> V_Log_Gate
- Q2 pad 2: GND -> V_In
- Q2 pad 3: Net-(Q2-Pad3) -> V_Out_Log
- R1 pad 1: CELL_1-GND_SENSE -> V_In
- R1 pad 2: CELL_1 -> Net-(D1-Pad2)
- R2 pad 1: CELL_1-GND_SENSE -> V_Out_Act
- R2 pad 2: GND -> Net-(D2-Pad2)
- R3 pad 1: CELL_2-1_SENSE -> V_Out_Log
- R3 pad 2: Net-(R3-Pad2) -> Net-(D3-Pad2)
- R4 pad 1: CELL_3-2_SENSE -> Net-(R4-Pad1)
- R4 pad 2: Net-(R4-Pad2) -> GND
- R5 pad 1: CELL_4-3_SENSE -> Net-(R5-Pad1)
- R5 pad 2: Net-(R5-Pad2) -> GND
- U1 pad 1: +3V3 -> V_In
- U1 pad 3: PACK_I_SENSE -> +3V3
- U2 pad 1: +5V -> GND
- U2 pad 2: Net-(Q1-Pad3) -> Net-(U2-Pad2)
- U3 pad 2: CELL_1 -> Net-(U3-Pad2)
- U3 pad 3: CELL_2 -> Net-(U3-Pad3)
- U3 pad 4: GND -> Net-(R5-Pad1)
- U3 pad 5: Net-(R3-Pad2) -> E-Stop_Gate
- U3 pad 6: Net-(R3-Pad2) -> V_In
- U3 pad 7: LOGIC_PWR -> (no net)
- U3 pad 8: Net-(U3-Pad8) -> V_In
- U4 pad 1: +5V -> Net-(R5-Pad1)
- U4 pad 2: Net-(Q4-Pad3) -> Net-(U4-Pad2)
- U5 pad 1: Net-(Q2-Pad3) -> Net-(U4-Pad2)
- U5 pad 2: +5V -> +3V3
- U5 pad 3: Net-(C10-Pad1) -> V_Out_Act
- U5 pad 4: Net-(F1-Pad2) -> GND
Routing:
- net +5V: track 450.7 -> 0.00 mm, vias 10 -> 0
- net LOGIC_PWR: track 292.8 -> 0.00 mm, vias 11 -> 0
- net V_OUT: track 226.3 -> 0.00 mm, vias 32 -> 0
- net /V_IN: track 212.2 -> 0.00 mm, vias 31 -> 0
- net +3V3: track 174.1 -> 0.00 mm, vias 2 -> 0
- net PACK_I_SENSE: track 163.6 -> 0.00 mm, vias 3 -> 0
- net Net-(R13-Pad1): track 147.0 -> 0.00 mm, vias 6 -> 0
- net SER_TX_IND: track 143.0 -> 0.00 mm, vias 4 -> 0
- net V_LOG_SENSE: track 121.6 -> 0.00 mm, vias 4 -> 0
- net CELL_8-7_SENSE: track 103.2 -> 0.00 mm, vias 2 -> 0
- net CELL_4: track 98.6 -> 0.00 mm, vias 2 -> 0
- net CELL_7-6_SENSE: track 94.0 -> 0.00 mm, vias 2 -> 0
- net CELL_5: track 92.8 -> 0.00 mm, vias 2 -> 0
- net Net-(Q2-Pad3): track 90.2 -> 0.00 mm, vias 2 -> 0
- net CELL_3: track 84.7 -> 0.00 mm, vias 1 -> 0
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- removed copper zone on B.Cu, net +3V3
- removed copper zone on F.Cu, net +3V3
- removed copper zone on F.Cu, net +5V
- removed copper zone on B.Cu, net /V_IN
- removed copper zone on F.Cu, net /V_IN
- removed copper zone on B.Cu, net GND
- removed copper zone on F.Cu, net GND
- removed copper zone on B.Cu, net Net-(C10-Pad1)
- removed copper zone on F.Cu, net Net-(C10-Pad1)
- removed copper zone on B.Cu, net Net-(F1-Pad2)
- removed copper zone on F.Cu, net Net-(F1-Pad2)
- removed copper zone on B.Cu, net V_OUT
- removed copper zone on F.Cu, net V_OUT
Other:
- board outline removed
- board text removed: "+"
- board text removed: "-"
- board text removed: "1"
- board text removed: "2"
- board text removed: "2-1"
- board text removed: "3"
- board text removed: "3-2"
- board text removed: "3V3 OKI"
- board text removed: "3v3"
- board text removed: "4"
- board text removed: "4-3"
- board text removed: "5"
- board text removed: "5-4"
- board text removed: "5V"
- board text removed: "5V OKI"
- board text removed: "6"
- board text removed: "6-5"
- board text removed: "7"
- board text removed: "7-6"
- board text removed: "8"
- board text removed: "8-7"
- board text removed: "BMS, REV. 2 MARS ROVER DESIGN TEAM MISSOURI S&T, 2019 Brian Dahlman"
- board text removed: "CHARGE SENSE"
- board text removed: "COIL"
- board text removed: "FAN CONTROL"
- board text removed: "GND"
- board text removed: "LED"
- board text removed: "LOG_PWR"
- board text removed: "SIG"
- board text removed: "SW_ERR"
- board text removed: "SW_IND"
- board text removed: "TX"
- board text removed: "V_IN"
- board text removed: "V_OUT"

Commit message: high level placement
Parts:
- moved U4 113.1 mm to (153.7, 94.0)
- moved U5 105.5 mm to (141.0, 94.0)
- moved Q1 89.6 mm to (180.3, 122.6), turned to 270 degrees
- moved U3 81.6 mm to (154.8, 127.6)
- moved C4 80.2 mm to (156.6, 116.8)
- moved Q2 78.3 mm to (167.6, 122.6), turned to 270 degrees
- moved R5 75.3 mm to (158.8, 93.1), turned to 90 degrees
- moved Conn1 71.3 mm to (128.5, 123.3)
- moved F1 69.2 mm to (197.0, 98.2)
- moved F2 69.2 mm to (197.0, 105.8)
- moved Conn2 68.6 mm to (206.8, 97.4)
- moved D3 63.6 mm to (195.8, 125.3), turned to 90 degrees
- moved D2 61.6 mm to (192.3, 125.3), turned to 90 degrees
- moved R3 58.1 mm to (195.8, 121.0), turned to 270 degrees
- moved SW1 56.8 mm to (167.8, 94.2), turned to 180 degrees
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Other:
- board text added: "+"
- board text added: "-"
- board text added: "20A"
- board text added: "5A"

Commit message: finished layout
Parts:
- added REF**: 6_32_Hole, MRDT_Drill_Holes:6_32_Hole_Corner, F.Cu at (214.0, 95.9)
- added REF**: 6_32_Hole, MRDT_Drill_Holes:6_32_Hole_Corner, F.Cu at (146.7, 95.9)
- added REF**: 6_32_Hole, MRDT_Drill_Holes:6_32_Hole_Corner, F.Cu at (146.7, 125.1)
- added REF**: 6_32_Hole, MRDT_Drill_Holes:6_32_Hole_Corner, F.Cu at (214.0, 125.1)
- moved C2 29.5 mm to (166.8, 114.3), turned to 180 degrees
- moved Conn1 25.4 mm to (153.9, 123.3)
- moved C1 25.2 mm to (163.4, 114.3), turned to 0 degrees
- moved C3 24.3 mm to (172.4, 113.5)
- moved U2 24.3 mm to (171.3, 103.5)
- moved U3 24.3 mm to (171.3, 109.9)
- moved C4 23.2 mm to (172.4, 99.8)
- moved U1 20.1 mm to (160.0, 115.6), turned to 0 degrees
- moved R5 18.2 mm to (165.0, 110.2), turned to 180 degrees
- moved R4 15.1 mm to (165.0, 107.7), turned to 180 degrees
- moved U5 14.8 mm to (153.7, 101.6)
- moved U4 13.7 mm to (142.2, 101.6)
- moved Q2 12.7 mm to (180.3, 122.6)
- moved Q1 12.7 mm to (193.0, 122.6)
- moved R2 12.6 mm to (204.5, 124.1)
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Routing:
- net V_Out_Act: track 0.00 -> 48.3 mm, vias 0 -> 17
- net +3V3: track 0.00 -> 41.2 mm, vias 0 -> 1
- net Net-(R5-Pad1): track 0.00 -> 38.4 mm
- net V_In: track 0.00 -> 38.2 mm, vias 0 -> 180
- net E-Stop_Gate: track 0.00 -> 33.5 mm
- net V_Out_Log: track 0.00 -> 27.9 mm, vias 0 -> 5
- net V_Log_Gate: track 0.00 -> 27.2 mm
- net Net-(R4-Pad1): track 0.00 -> 12.2 mm
- net Net-(U4-Pad2): track 0.00 -> 6.35 mm
- net Net-(D3-Pad2): track 0.00 -> 2.06 mm
- net Net-(D2-Pad2): track 0.00 -> 2.06 mm
- net Net-(D1-Pad2): track 0.00 -> 2.06 mm
- added copper zone on B.Cu, net GND
- added copper zone on F.Cu, net GND
- added copper zone on B.Cu, net Net-(Conn2-Pad2)
- added copper zone on F.Cu, net Net-(Conn2-Pad2)
- added copper zone on B.Cu, net Net-(Conn2-Pad3)
- added copper zone on F.Cu, net Net-(Conn2-Pad3)
- added copper zone on B.Cu, net V_In
- added copper zone on F.Cu, net V_In
- added copper zone on B.Cu, net V_Out_Act
- added copper zone on F.Cu, net V_Out_Act
- added copper zone on B.Cu, net V_Out_Log
- added copper zone on F.Cu, net V_Out_Log
Other:
- board outline added: 86.4 x 48.3 mm
- board text added: "Act"
- board text added: "Log"
- board text added: "V In"

Commit message: switched logic pushbutton to be NO
Parts:
- added G***: LOGO, MRDT_Silkscreens:z_sig_Andrew_Van_Horn_Sig_15mm, F.Cu at (205.7, 91.4)
- moved Logic 52.9 mm to (210.8, 127.0)
- moved R4 0.13 mm to (165.0, 107.6), turned to 0 degrees
- renumbered SW1 to Logic
Connections:
- Logic pad 1: Net-(R4-Pad1) -> Net-(R4-Pad2)
- Logic pad 2: +3V3 -> GND
- R4 pad 1: Net-(R4-Pad1) -> +3V3
- R4 pad 2: GND -> Net-(R4-Pad2)
- U2 pad 4: Net-(R4-Pad1) -> Net-(R4-Pad2)
Routing:
- net Net-(R4-Pad2): track 0.00 -> 95.3 mm, vias 0 -> 2
- net Net-(R4-Pad1): track 12.2 -> 0.00 mm
- net V_Out_Act: track 48.3 -> 45.4 mm
- net +3V3: track 41.2 -> 39.9 mm
- net Net-(R5-Pad1): track 38.4 -> 39.2 mm
Other:
- board text added: "E-Stop Board, Rev1 Mars Rover Design Team Missouri S&T, 2020 Andrew Van Horn"

Commit message: Final changes before PRR
Parts:
- removed the REF** at (214.0, 95.9)
- removed the REF** at (146.7, 95.9)
- removed the REF** at (146.7, 125.1)
- removed the REF** at (214.0, 125.1)
- added REF**: 4_40_Hole, MRDT_Drill_Holes:4_40_Hole_Corner, F.Cu at (214.4, 125.5)
- added REF**: 4_40_Hole, MRDT_Drill_Holes:4_40_Hole_Corner, F.Cu at (146.2, 125.5)
- added REF**: 4_40_Hole, MRDT_Drill_Holes:4_40_Hole_Corner, F.Cu at (146.2, 95.4)
- added REF**: 4_40_Hole, MRDT_Drill_Holes:4_40_Hole_Corner, F.Cu at (214.4, 95.4)
- moved G*** 28.1 mm to (177.8, 94.0)
- moved Logic 2.60 mm to (210.6, 124.5), turned to 0 degrees
- moved D2 1.27 mm to (204.5, 126.6)
- moved D3 1.27 mm to (201.9, 126.6)
- moved R2 1.27 mm to (204.5, 122.8)
- moved R3 1.27 mm to (201.9, 122.8)
Routing:
- net Net-(R4-Pad2): track 95.3 -> 89.3 mm
- net V_Out_Log: track 27.9 -> 26.1 mm
Other:
- board size 86.4 x 48.3 mm -> 84.3 x 46.2 mm
- board text added: "A"
- board text added: "D"
- board text added: "G"
- board text added: "L"

Commit message: created gerbs
Parts:
- removed U4: E_STOP, MRDT_Connectors:MOLEX_SL_02_Vertical
- added G***: LOGO, MRDT_Silkscreens:0_MRDT_Logo_40mm, B.Cu at (178.1, 111.0)
Connections:
- net E-Stop_Gate renamed V_Act_Gate
- net V_In renamed +12V
- net V_Out_Act renamed +12VA
- net V_Out_Log renamed +12L
- U5 pad 1: Net-(U4-Pad2) -> Net-(R5-Pad1)
Routing:
- net Net-(R5-Pad1): track 39.2 -> 30.3 mm
- net Net-(U4-Pad2): track 6.35 -> 0.00 mm
- net +12VA: track 45.8 -> 48.1 mm
- net GND: vias 0 -> 69
Other:
- board text added: "Arm E-Stop Board, Rev1 Mars Rover Design Team Missouri S&T, 2020 Andrew Van Horn"
- board text added: "Logic Stop"
- board text removed: "E-Stop Board, Rev1 Mars Rover Design Team Missouri S&T, 2020 Andrew Van Horn"
